File: PROJET_GAM/PROJET_GAM.kicad_sch (KiCad schematic)
At the start: 0 parts

Commit message: Schéma Premiere version
Parts:
- added C1, C2: 690n, 0_myfootprint:C_Disc_D3.0mm_W1.6mm_P2.50mm, symbol Device:C
- added C10: 82n, symbol Device:C
- added C11, C8: 22u, symbol Device:C
- added C12: 1uF, symbol Device:C
- added C3, C4: 100n, 0_myfootprint:C_Disc_D3.0mm_W1.6mm_P2.50mm, symbol Device:C
- added C5, C6, C7: 100n, symbol Device:C
- added C9: 22p, symbol Device:C
- added D1, D2, D3: 1N4001, Diode_THT:D_DO-41_SOD81_P10.16mm_Horizontal, symbol Diode:1N4001
- added J1, J10, J3, J4, J5, J6, J7, J8, J9: Conn_01x01_Pin, 0_myfootprint:PinHeader_1x01_P1.00mm_Vertical, symbol Connector:Conn_01x01_Pin
- added J11: Conn_01x02, symbol Connector_Generic:Conn_01x02
- added J2: Conn_01x03, symbol Connector_Generic:Conn_01x03
- added Q1: BC547, Package_TO_SOT_THT:TO-92_Inline, symbol Transistor_BJT:BC547
- added Q2: BS170, Package_TO_SOT_THT:TO-92_Inline, symbol Transistor_FET:BS170
- added R1, R10, R11, R14, R15, R2, R3, R6, R7, R8: 10k, 0_myfootprint:R_Axial_DIN0204_L3.6mm_D1.6mm_P5.08mm_Horizontal, symbol Device:R
- added R12: 1.8M, 0_myfootprint:R_Axial_DIN0204_L3.6mm_D1.6mm_P5.08mm_Horizontal, symbol Device:R
- added R13: 3.3M, 0_myfootprint:R_Axial_DIN0204_L3.6mm_D1.6mm_P5.08mm_Horizontal, symbol Device:R
- added R16, R17, R18, R20, R21, R22, R25, R26, R39, R48, R52, R54, R55, R60: 1k, symbol Device:R
- added R19, R24, R40, R42, R46: 100k, symbol Device:R
- added R23, R28, R29, R34, R35, R36, R41, R43, R44, R47, R58: 10k, symbol Device:R
- added R27: 750, symbol Device:R
- added R30: 8590, symbol Device:R
- added R31, R32: 1.8k, symbol Device:R
- added R33: 140k, symbol Device:R
- added R37: 50, symbol Device:R
- added R38: 25k, symbol Device:R
- added R4: 100k, 0_myfootprint:R_Axial_DIN0204_L3.6mm_D1.6mm_P5.08mm_Horizontal, symbol Device:R
- added R45: 2k, symbol Device:R
- added R49, R57: 20k, symbol Device:R
- added R5, R9: 5k, 0_myfootprint:R_Axial_DIN0204_L3.6mm_D1.6mm_P5.08mm_Horizontal, symbol Device:R
- added R50, R53, R59: 3.3k, symbol Device:R
- added R51, R56: 1K, symbol Device:R
- added R61: 6.2k, symbol Device:R
- added RV1, RV2: 1k, symbol Device:R_Potentiometer
- added RV3: 1M, symbol Device:R_Potentiometer
- added SW1: SW_Push, symbol Switch:SW_Push
- added U1, U10, U11, U14, U15, U16, U2, U3, U4, U5, U6: TL072, symbol Amplifier_Operational:TL072
- added U12, U13: TL071, symbol Amplifier_Operational:TL071
- added U17, U8, U9: LCC110, Package_DIP:DIP-8_W7.62mm, symbol Relay_SolidState:LCC110
Connections:
- new net: R50.1, R53.1, R56.2, R59.1, U15.6 (-)
- new net: R59.2, U15.1
- new net: C7.2, R21.1, R24.1, U5.1
- new net: R24.2, R25.2, R26.1, U6.6 (-)
- new net: C1.2, J7.1 (Pin_1), R12.2, RV3.3, U2.7
- new net: C2.2, J8.1 (Pin_1), R13.1, R14.1, U3.1
- new net: R44.1, R45.2, U13.3 (+)
- new net: R31.1, U9.2
- new net: Q1.1 (C), U8.3, U9.3
- new net: J3.1 (Pin_1), R1.2, R4.1, U1.1
- new net: R4.2, R6.2, U1.6 (-)
- new net: R51.1, U15.5 (+)
- new net: R56.1, U14.3 (+), U15.7
- new net: J9.1 (Pin_1), R15.1, U3.7, U4.5 (+)
- new net: R14.2, R15.2, U3.6 (-)
- new net: C10.1, U6.1
- new net: C11.2, R41.1, U6.2 (-)
- new net: R42.1, U6.3 (+)
- new net: C6.1, R21.2, U5.6 (-)
- new net: C6.2, R18.2, R19.1, U5.7
- new net: C9.1, D2.2 (A), R35.1, U10.2 (-)
- new net: R35.2, R36.1, U11.6 (-)
- new net: C2.1, R12.1, R13.2, U3.2 (-)
- new net: R17.2, R19.2, R20.1, U4.2 (-)
- new net: R16.2, U4.3 (+)
- new net: C10.2, R39.1
- new net: R37.1, R39.2, U10.6 (-)
- new net: R2.2, R3.1, U1.3 (+)
- new net: J1.1 (Pin_1), R3.2, RV1.2
- new net: D3.1 (K), R47.2, U11.5 (+)
- new net: C9.2, D2.1 (K), D3.2 (A), U10.1
- new net: R50.2, U11.1
- new net: R48.2, R49.2, U11.3 (+)
- new net: R60.2, R61.2, U15.2 (-)
- new net: C7.1, R23.2, U5.2 (-)
- new net: R29.2, R30.1, U14.5 (+)
- new net: D1.2 (A), J5.1 (Pin_1), R10.2, RV2.1, U2.1
- new net: J6.1 (Pin_1), R8.1, RV2.2
- new net: R37.2, U10.3 (+), U10.7
- new net: R1.1, U1.2 (-)
- new net: R36.2, U11.7, U13.2 (-)
- new net: R40.1, R44.2, U13.6
- new net: Q2.1 (D), U17.3
- new net: Q2.2 (G), U14.1
- new net: R54.2, R57.2, U16.6 (-)
- new net: R27.2, R28.1, R29.1, U14.7
- new net: Q1.2 (B), R28.2
- new net: R22.2, U6.5 (+)
- new net: R55.2, R58.2, U14.2 (-)
- new net: R52.2, U17.2
- new net: D1.1 (K), R7.1, R8.2, U2.2 (-)
- new net: C5.1, R18.1, U5.3 (+)
- new net: R9.2, U2.3 (+)
- new net: C8.2, R27.1, U14.6 (-)
- new net: R40.2, R46.1, U12.2 (-)
- new net: C11.1, J11.1 (Pin_1)
- new net: R5.2, U1.5 (+)
- new net: J4.1 (Pin_1), R6.1, R7.2, U1.7
- new net: R38.1, R46.2, U12.6
- new net: R32.2, U8.2
- new net: R33.2, R34.1, U12.3 (+)
- new net: C1.1, R10.1, R11.1, RV3.2, U2.6 (-)
- new net: C12.1, U17.6, U17.7
- new net: R53.2, U16.7
- new net GND: C12.2, C3.1, C4.2, C5.2, C8.1, J11.2 (Pin_2), J2.2 (Pin_2), Q1.3 (E), Q2.3 (S), R16.1, R22.1, R23.1, R30.2, R34.2, R41.2, R42.2, R43.1, R45.1, R47.1, R49.1, R5.1, R51.2, R57.1, R58.1, R61.1, R9.1, RV1.3, RV2.3, RV3.1, U10.5 (+), U13.4 (V-), U2.5 (+), U3.3 (+), U3.5 (+), U5.5 (+)
- new net Vcc: C3.2, J2.1 (Pin_1), R31.2, R32.1, R33.1, R48.1, R52.1, R54.1, R55.1, R60.1, RV1.1, SW1.1, U1.8 (V+), U10.8 (V+), U11.8 (V+), U12.7 (V+), U13.7 (V+), U14.8 (V+), U15.8 (V+), U16.8 (V+), U2.8 (V+), U3.8 (V+), U4.8 (V+), U5.8 (V+)
- new net Vee: C4.1, J2.3 (Pin_3), U1.4 (V-), U10.4 (V-), U11.4 (V-), U12.4 (V-), U14.4 (V-), U15.4 (V-), U16.4 (V-), U2.4 (V-), U3.4 (V-), U4.4 (V-), U5.4 (V-)
- new net Vin_button: R11.2, SW1.2
- new net X_position: R17.1, R38.2, R43.2, U11.2 (-), U16.5 (+), U17.8
- new net X_trigger: U17.5
- new net Y_position: J10.1 (Pin_1), R2.1, R25.1, U15.3 (+), U4.6 (-), U4.7
- new net gen_balle_X: R20.2, U4.1, U8.6
- new net gen_balle_Y: R26.2, U6.7, U9.6
- new net gen_terr_X: U8.8
- new net gen_terr_Y: U9.8
- new net out_X: U8.5, U8.7
- new net out_Y: U9.5, U9.7
Other:
- note added: "ALIMENTATION"
- note added: "BUTTON"
- note added: "DEPLACEMENT X"
- note added: "DEPLACEMENT Y"
- note added: "GENERATION BALLE"
- note added: "HIT NET"
- note added: "INTEGRATEUR_1"
- note added: "INTEGRATEUR_2"
- note added: "INTEGRATION AFFICHAGE"
- note added: "INVERSEUR"
- note added: "INVERTER"
- note added: "OFFSET"
- note added: "REDRESSEUR"
- note added: "YA QUOI ICI ?"
